File: CAD/Thermorad-C.sch (EAGLE design)
At the start: 84 parts, among them IC1 LM324D, IC2 TPS61070DDC, IC4 LM324D, J1 DNP, SW1 450404015514, SW2 450404015514, T1 DNP, U1 ADL5910, U2 LM2936M-3.3, U3 LM2936M-5.0/DNP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

Commit message: Update C - Cheaper Potentiometer implanted
Parts:
- C1: value CBF/0805/742792037 -> CSGP/0805/1µF/885012107015
- C11, C13: value 1N4148 -> DNP/1N4148
- C9: value !RES/0805/82R -> DNP/!RES/0805/82R
- L1: value CAP/0805/470pF/NP0 -> RES/0805/82R/5%
- L2: value RES/0805/1k -> RES/0805/10k
- R10, R11: value 10k -> 2k2
- R15: value 1K -> 10k
- R16, R17: value 1k -> 10k
- R18: device rcl:R-EU_R0603 -> resistor:R-EU_M0805
- R21, R22, R23: value 0603/10k -> 10k; device rcl:R-EU_R0603 -> resistor:R-EU_M0805
- SHC1: value 36103205S -> DNP/36103205S
- X1: value BU-SMA-V -> DNP/BU-SMA-V
Connections:
- net +3V3: now also R21.1; no longer R21.2
- net N$36: now also R21.2; no longer R21.1
- net VDD: now also C7.2, U2.VIN
- net VEE: no longer C7.2, U2.VIN
Other:
- moved on the sheet: R21
